File: cad/MagicMatrix/MagicMatrix.kicad_sch (KiCad schematic)
At the start: 5 parts, among them SW1 Reset, U1 Raspberry Pi Pico

Commit message: update
Parts:
- added IRM-3638T: 红外线接收模块, OptoDevice:Vishay_MINIMOLD-3Pin, symbol Interface_Optical:TSOP21xx
- WS2812B: renamed from D1; value WS2812B -> RGB矩阵模块
Connections:
- net GND: now also IRM-3638T.3 (GND)
- net VSYS: now also IRM-3638T.2 (Vs)
- new net GPIO22: IRM-3638T.1 (OUT)
Other:
- company: (none) -> DXEdu
- title: (none) -> MagicMatrix
Changed lines of the file:
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@@
 (kicad_sch (version 20230121) (generator eeschema)
   (paper "A4")
+  (title_block
+    (title "MagicMatrix")
+    (date "2024-02-13")
+    (company "DXEdu")
+  )
   (junction (at 88.9 49.53) (diameter 0) (color 0 0 0 0)
   )
@@
     (stroke (width 0) (type default))
   )
+  (wire (pts (xy 203.2 83.82) (xy 210.82 83.82))
+    (stroke (width 0) (type default))
+  )
   (wire (pts (xy 135.89 39.37) (xy 144.78 39.37))
     (stroke (width 0) (type default))
@@
     (stroke (width 0) (type default))
   )
+  (wire (pts (xy 203.2 78.74) (xy 210.82 78.74))
+    (stroke (width 0) (type default))
+  )
   (wire (pts (xy 88.9 52.07) (xy 88.9 49.53))
     (stroke (width 0) (type default))
@@
     (stroke (width 0) (type default))
   )
+  (wire (pts (xy 203.2 73.66) (xy 210.82 73.66))
+    (stroke (width 0) (type default))
+  )
   (wire (pts (xy 234.95 26.67) (xy 234.95 30.48))
     (stroke (width 0) (type default))
@@
     (stroke (width 0) (type default))
   )
+  (label "GPIO22" (at 203.2 78.74 0) (fields_autoplaced)
+    (effects (font (size 1.27 1.27)) (justify left bottom))
+  )
   (label "VSYS" (at 152.4 26.67 0) (fields_autoplaced)
     (effects (font (size 1.27 1.27)) (justify left bottom))
@@
     (effects (font (size 1.27 1.27)) (justify left bottom))
   )
+  (label "VSYS" (at 203.2 73.66 0) (fields_autoplaced)
+    (effects (font (size 1.27 1.27)) (justify left bottom))
+  )
   (label "GPIO21" (at 135.89 39.37 0) (fields_autoplaced)
     (effects (font (size 1.27 1.27)) (justify left bottom))
@@
   (label "GPIO2" (at 218.44 38.1 0) (fields_autoplaced)
     (effects (font (size 1.27 1.27)) (justify left bottom))
+  )
+  (symbol (lib_id "Interface_Optical:TSOP21xx") (at 220.98 78.74 0) (mirror y) (unit 1)
+    (in_bom yes) (on_board yes) (dnp no)
+    (property "Reference" "IRM-3638T" (at 233.68 80.01 0)
+      (effects (font (size 1.27 1.27)) (justify right))
+    )
+    (property "Value" "红外线接收模块" (at 233.68 77.47 0)
+      (effects (font (size 1.27 1.27)) (justify right))
+    )
+    (property "Footprint" "OptoDevice:Vishay_MINIMOLD-3Pin" (at 222.25 88.265 0)
+      (effects (font (size 1.27 1.27)) hide)
+    )
+    (property "Datasheet" "http://www.vishay.com/docs/82460/tsop45.pdf" (at 204.47 71.12 0)
+      (effects (font (size 1.27 1.27)) hide)
+    )
+    (pin "2")
+    (pin "1")
+    (pin "3")
+    (instances
+      (project "MagicMatrix"
+        (path "/b8e9c7d0-a14a-432a-8356-23b1463ea8e9"
+          (reference "IRM-3638T") (unit 1)
+        )
+      )
+    )
   )
   (symbol (lib_id "power:GNDREF") (at 181.61 38.1 0) (unit 1)
@@
     )
   )
+  (symbol (lib_id "power:GNDREF") (at 203.2 83.82 0) (unit 1)
+    (in_bom yes) (on_board yes) (dnp no) (fields_autoplaced)
+    (property "Reference" "#PWR08" (at 203.2 90.17 0)
+      (effects (font (size 1.27 1.27)) hide)
+    )
+    (property "Value" "GNDREF" (at 203.2 88.9 0)
+      (effects (font (size 1.27 1.27)))
+    )
+    (property "Footprint" "" (at 203.2 83.82 0)
+      (effects (font (size 1.27 1.27)) hide)
+    )
+    (property "Datasheet" "" (at 203.2 83.82 0)
+      (effects (font (size 1.27 1.27)) hide)
+    )
+    (pin "1")
+    (instances
+      (project "MagicMatrix"
+        (path "/b8e9c7d0-a14a-432a-8356-23b1463ea8e9"
+          (reference "#PWR08") (unit 1)
+        )
+      )
+    )
+  )
   (symbol (lib_id "power:GND") (at 88.9 38.1 180) (unit 1)
     (in_bom yes) (on_board yes) (dnp no) (fields_autoplaced)
@@
   (symbol (lib_id "LED:WS2812B") (at 234.95 38.1 0) (unit 1)
     (in_bom yes) (on_board yes) (dnp no) (fields_autoplaced)
-    (property "Reference" "D1" (at 246.38 34.4521 0)
-      (effects (font (size 1.27 1.27)))
-    )
-    (property "Value" "WS2812B" (at 246.38 36.9921 0)
+    (property "Reference" "WS2812B" (at 246.38 34.4521 0)
+      (effects (font (size 1.27 1.27)))
+    )
+    (property "Value" "RGB矩阵模块" (at 246.38 36.9921 0)
       (effects (font (size 1.27 1.27)))
     )
@@
       (project "MagicMatrix"
         (path "/b8e9c7d0-a14a-432a-8356-23b1463ea8e9"
-          (reference "D1") (unit 1)
-        )
-      )
+          (reference "WS2812B") (unit 1)
+        )
+      )

Commit message: update
Parts:
- added PIR1: 红外线人体探测模块, symbol MCU_RaspberryPi_and_Boards:PIR
Connections:
- net GND: now also PIR1.3 (GND)
- net VSYS: now also PIR1.1 (VDD)
- new net GPIO7: PIR1.2 (OUT)
Other:
- moved on the sheet: BZ1, IRM-3638T, SW1, U1, WS2812B, 温湿度传感器
