File: cad/MagicMatrix/MagicMatrix.kicad_sch (KiCad schematic)
At the start: 7 parts, among them SW1 Reset, U1 Raspberry Pi Pico

Commit message: update
Parts:
- removed 温湿度传感器: DHT11, Sensor:Aosong_DHT11_5.5x12.0_P2.54mm, symbol Sensor:DHT11
- added DHT11_1: 温湿度传感器, Sensor:Aosong_DHT11_5.5x12.0_P2.54mm, symbol MagicMatrix:DHT11
- IRM_1: renamed from IRM-3638T; footprint OptoDevice:Vishay_MINIMOLD-3Pin -> OptoDevice:Vishay_MOLD-3Pin; symbol Interface_Optical:TSOP21xx -> MagicMatrix:TSOP21xx
- PIR1: symbol MCU_RaspberryPi_and_Boards:PIR -> MagicMatrix:PIR
- U1: footprint RPi_Pico:RPi_Pico_SMD_TH -> RP2040; symbol MCU_RaspberryPi_and_Boards:Pico -> MagicMatrix:Pico
- renumbered BZ1 to BZ_1, SW1 to SW_1, WS2812B to WS2812B_1
Connections:
- net GPIO2: now also U1.4 (GPIO2)
- net GPIO20: now also U1.26 (GPIO20)
- net GPIO21: now also U1.27 (GPIO21), DHT11_1.2 (DATA)
- net GPIO22: now also U1.29 (GPIO22)
- net GPIO7: now also U1.10 (GPIO7)
- net VSYS: now also U1.39 (VSYS), DHT11_1.1 (VDD)
- net RUN: now reaches SW_1.1, U1.30 (RUN)
- net +5V: no longer names the net of U1.40 (VBUS)
- net GND renamed GNDREF
- net GNDREF: now also DHT11_1.4 (GND)
- no-connect marks 0 -> 20
Other:
- moved on the sheet: IRM_1, SW_1

Commit message: update
Parts:
- PIR1: footprint (none) -> Connector_PinSocket_1.27mm:PinSocket_1x03_P1.27mm_Vertical
- SW_1: footprint (none) -> Connector_PinHeader_2.54mm:PinHeader_2x02_P2.54mm_Vertical_SMD
- U1: footprint RP2040 -> MCU_RaspberryPi_and_Boards:RPi_Pico_SMD_TH; symbol MagicMatrix:Pico -> MCU_RaspberryPi_and_Boards:Pico
Changed lines of the file:
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@@
       (effects (font (size 1.27 1.27)) (justify left))
     )
-    (property "Footprint" "" (at 114.3 67.31 0)
+    (property "Footprint" "Connector_PinSocket_1.27mm:PinSocket_1x03_P1.27mm_Vertical" (at 114.3 67.31 0)
       (effects (font (size 1.27 1.27)) hide)
     )
@@
     )
   )
-  (symbol (lib_id "MagicMatrix:Pico") (at 44.45 54.61 0) (unit 1)
+  (symbol (lib_id "MCU_RaspberryPi_and_Boards:Pico") (at 44.45 54.61 0) (unit 1)
     (in_bom yes) (on_board yes) (dnp no) (fields_autoplaced)
     (property "Reference" "U1" (at 44.45 22.86 0)
@@
       (effects (font (size 1.27 1.27)))
     )
-    (property "Footprint" "RP2040" (at 44.45 54.61 90)
+    (property "Footprint" "MCU_RaspberryPi_and_Boards:RPi_Pico_SMD_TH" (at 44.45 54.61 90)
       (effects (font (size 1.27 1.27)) hide)
     )
@@
       (effects (font (size 1.27 1.27)))
     )
-    (property "Footprint" "" (at 168.91 71.12 0)
-      (effects (font (size 1.27 1.27)) hide)
-    )
+    (property "Footprint" "Connector_PinHeader_2.54mm:PinHeader_2x02_P2.54mm_Vertical_SMD" (at 168.91 71.12 0)
+      (effects (font (size 1.27 1.27)) hide)
+    )

Commit message: update
Parts:
- removed WS2812B_1: RGB矩阵模块, LED_SMD:LED_WS2812B_PLCC4_5.0x5.0mm_P3.2mm, symbol LED:WS2812B
- added WSM1: ~, symbol MagicMatrix:WS2812Matrix
Connections:
- net GNDREF: now also WSM1. (VCC)
- net VSYS: now also WSM1. (VCC)
- no-connect marks 20 -> 19
Changed lines of the file:
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@@
-	)
-	(no_connect
-		(at 213.36 40.64)
 	)
 	(no_connect
@@
 	(wire
 		(pts
-			(xy 189.23 40.64) (xy 198.12 40.64)
-		)
-		(stroke
-			(width 0)
-			(type default)
-		)
-	)
-	(wire
-		(pts
 			(xy 105.41 48.26) (xy 111.76 48.26)
 		)
@@
 	(wire
 		(pts
+			(xy 193.04 39.37) (xy 199.39 39.37)
+		)
+		(stroke
+			(width 0)
+			(type default)
+		)
+	)
+	(wire
+		(pts
 			(xy 152.4 38.1) (xy 161.29 38.1)
 		)
@@
 	(wire
 		(pts
+			(xy 193.04 34.29) (xy 199.39 34.29)
+		)
+		(stroke
+			(width 0)
+			(type default)
+		)
+	)
+	(wire
+		(pts
 			(xy 229.87 35.56) (xy 240.03 35.56)
 		)
@@
 		(pts
 			(xy 101.6 76.2) (xy 109.22 76.2)
-		)
-		(stroke
-			(width 0)
-			(type default)
-		)
-	)
-	(wire
-		(pts
-			(xy 205.74 29.21) (xy 205.74 33.02)
-		)
-		(stroke
-			(width 0)
-			(type default)
-		)
-	)
-	(wire
-		(pts
-			(xy 205.74 48.26) (xy 205.74 52.07)
 		)
 		(stroke
@@
 		)
 	)
-	(label "VSYS"
-		(at 205.74 29.21 0)
-		(fields_autoplaced yes)
-		(effects
-			(font
-				(size 1.27 1.27)
-			)
-			(justify left bottom)
-		)
-	)
 	(label "GPIO7"
 		(at 101.6 76.2 0)
@@
 	)
 	(label "VSYS"
+		(at 193.04 34.29 0)
+		(fields_autoplaced yes)
+		(effects
+			(font
+				(size 1.27 1.27)
+			)
+			(justify left bottom)
+		)
+	)
+	(label "VSYS"
 		(at 101.6 71.12 0)
 		(fields_autoplaced yes)
@@
 	(label "GPIO20"
 		(at 67.31 66.04 0)
-		(fields_autoplaced yes)
-		(effects
-			(font
-				(size 1.27 1.27)
-			)
-			(justify left bottom)
-		)
-	)
-	(label "GPIO2"
-		(at 189.23 40.64 0)
 		(fields_autoplaced yes)
 		(effects
@@
 	)
 	(symbol
+		(lib_name "GNDREF_1")
+		(lib_id "power:GNDREF")
+		(at 193.04 39.37 0)
+		(unit 1)
+		(exclude_from_sim no)
+		(in_bom yes)
+		(on_board yes)
+		(dnp no)
+		(fields_autoplaced yes)
+		(property "Reference" "#PWR01"
+			(at 193.04 45.72 0)
+			(effects
+				(font
+					(size 1.27 1.27)
+				)
+				(hide yes)
+			)
+		)
+		(property "Value" "GNDREF"
+			(at 193.04 44.45 0)
+			(effects
+				(font
+					(size 1.27 1.27)
+				)
+			)
+		)
+		(property "Footprint" ""
+			(at 193.04 39.37 0)
+			(effects
+				(font
+					(size 1.27 1.27)
+				)
+				(hide yes)
+			)
+		)
+		(property "Datasheet" ""
+			(at 193.04 39.37 0)
+			(effects
+				(font
+					(size 1.27 1.27)
+				)
+				(hide yes)
+			)
+		)
+		(property "Description" "Power symbol creates a global label with name \"GNDREF\" , reference supply ground"
+			(at 193.04 39.37 0)
+			(effects
+				(font
+					(size 1.27 1.27)
+				)
+				(hide yes)
+			)
+		)
+		(pin "1"
+		)
+		(instances
+			(project "MagicMatrix"
+				(path "/b8e9c7d0-a14a-432a-8356-23b1463ea8e9"
+					(reference "#PWR01")
+					(unit 1)
+				)
+			)
+		)
+	)
+	(symbol
+		(lib_id "MagicMatrix:WS2812Matrix")
+		(at 204.47 36.83 0)
+		(unit 1)
+		(exclude_from_sim no)
+		(in_bom yes)
+		(on_board yes)
+		(dnp no)
+		(fields_autoplaced yes)
+		(property "Reference" "WSM1"
+			(at 213.36 36.1949 0)
+			(effects
+				(font
+					(size 1.27 1.27)
+				)
+				(justify left)
+			)
+		)
+		(property "Value" "~"
+			(at 213.36 38.1 0)
+			(effects
+				(font
+					(size 1.27 1.27)
+				)
+				(justify left)
+			)
+		)
+		(property "Footprint" ""
+			(at 204.47 36.83 0)
+			(effects
+				(font
+					(size 1.27 1.27)
+				)
+				(hide yes)
+			)
+		)
+		(property "Datasheet" ""
+			(at 204.47 36.83 0)
+			(effects
+				(font
+					(size 1.27 1.27)
+				)
+				(hide yes)
+			)
+		)
+		(property "Description" "WS2812矩阵屏幕接口"
+			(at 203.2 43.18 0)
+			(effects
+				(font
+					(size 1.27 1.27)
+				)
+				(hide yes)
+			)
+		)
+		(pin ""
+		)
+		(pin ""
+		)
+		(pin ""
+		)
+		(instances
+			(project "MagicMatrix"
+				(path "/b8e9c7d0-a14a-432a-8356-23b1463ea8e9"
+					(reference "WSM1")
+					(unit 1)
+				)
+			)
+		)
+	)
+	(symbol
 		(lib_id "power:GNDREF")
 		(at 152.4 43.18 0)
@@
 	(symbol
 		(lib_id "power:GNDREF")
-		(at 205.74 52.07 0)
-		(unit 1)
-		(exclude_from_sim no)
-		(in_bom yes)
-		(on_board yes)
-		(dnp no)
-		(fields_autoplaced yes)
-		(property "Reference" "#PWR05"
-			(at 205.74 58.42 0)
-			(effects
-				(font
-					(size 1.27 1.27)
-				)
-				(hide yes)
-			)
-		)
-		(property "Value" "GNDREF"
-			(at 205.74 57.15 0)
-			(effects
-				(font
-					(size 1.27 1.27)
-				)
-			)
-		)
-		(property "Footprint" ""
-			(at 205.74 52.07 0)
-			(effects
-				(font
-					(size 1.27 1.27)
-				)
-				(hide yes)
-			)
-		)
-		(property "Datasheet" ""
-			(at 205.74 52.07 0)
-			(effects
-				(font
-					(size 1.27 1.27)
-				)
-				(hide yes)
-			)
-		)
-		(property "Description" ""
-			(at 205.74 52.07 0)
-			(effects
-				(font
-					(size 1.27 1.27)
-				)
-				(hide yes)
-			)
-		)
-		(pin "1"
-		)
-		(instances
-			(project "MagicMatrix"
-				(path "/b8e9c7d0-a14a-432a-8356-23b1463ea8e9"
-					(reference "#PWR05")
-					(unit 1)
-				)
-			)
-		)
-	)
-	(symbol
-		(lib_id "power:GNDREF")
 		(at 101.6 81.28 0)
 		(unit 1)
@@
 					(unit 1)
 				)
-			)
-		)
-	)
-	(symbol
-		(lib_id "LED:WS2812B")
-		(at 205.74 40.64 0)
-		(unit 1)
-		(exclude_from_sim no)
-		(in_bom yes)
-		(on_board yes)
-		(dnp no)
-		(property "Reference" "WS2812B_1"
-			(at 218.44 34.29 0)
-			(effects
-				(font
-					(size 1.27 1.27)
-				)
-			)
-		)
-		(property "Value" "RGB矩阵模块"
-			(at 218.44 36.83 0)
-			(effects
-				(font
-					(size 1.27 1.27)
-				)
-			)
-		)
-		(property "Footprint" "LED_SMD:LED_WS2812B_PLCC4_5.0x5.0mm_P3.2mm"
-			(at 207.01 48.26 0)
-			(effects
-				(font
-					(size 1.27 1.27)
-				)
-				(justify left top)
-				(hide yes)
-			)
-		)
-		(property "Datasheet" "https://cdn-shop.adafruit.com/datasheets/WS2812B.pdf"
-			(at 208.28 50.165 0)
-			(effects
-				(font
-					(size 1.27 1.27)
-				)
-				(justify left top)
-				(hide yes)
-			)
-		)
-		(property "Description" ""
-			(at 205.74 40.64 0)
-			(effects
-				(font
-					(size 1.27 1.27)
-				)
-				(hide yes)
-			)
-		)
-		(pin "1"
-		)
-		(pin "3"
-		)
-		(pin "2"
-		)
-		(pin "4"
-		)
-		(instances
-			(project "MagicMatrix"
-				(path "/b8e9c7d0-a14a-432a-8356-23b1463ea8e9"
-					(reference "WS2812B_1")
-					(unit 1)
-				)
