File: cad/MagicMatrix/MagicMatrix.kicad_pcb (KiCad board)
At the start: 2 copper layers, 0 parts

Commit message: update
Parts:
- added DHT11_1: 温湿度传感器, Sensor:Aosong_DHT11_5.5x12.0_P2.54mm, F.Cu at (99.5, 48.5)
- added IRM_1: 红外线接收模块, OptoDevice:Vishay_MOLD-3Pin, F.Cu at (94.9, 93.5)
- added PIR1: 红外线人体探测模块, Connector_PinSocket_1.27mm:PinSocket_1x03_P1.27mm_Vertical, F.Cu at (100.0, 79.2)
- added SW_1: Reset, Connector_PinHeader_2.54mm:PinHeader_2x02_P2.54mm_Vertical_SMD, F.Cu at (102.5, 69.8)
- added U1: Raspberry Pi Pico, MCU_RaspberryPi_and_Boards:RPi_Pico_SMD_TH, F.Cu at (76.6, 70.1)
